File: template/mlab-default/mlab-default.kicad_sch (KiCad schematic)
At the start: 8 parts, among them J1 Umin ... Umax, M1 HOLE, M2 HOLE, M3 HOLE, M4 HOLE

Commit message: Update module template.
Parts:
- removed C1: C/U, symbol mlab-default-rescue:CP2
- removed C2: 100nF, symbol mlab-default-rescue:C
- removed D1: DIODE, symbol mlab-default-rescue:DIODE
- added C1: 10uF, Capacitor_SMD:C_0805_2012Metric, symbol ISM02A-rescue:C_Small-Device-ISM02A-rescue
- added C2: 100nF, Capacitor_SMD:C_0805_2012Metric, symbol ISM02A-rescue:C_Small-Device-ISM02A-rescue
- added D1: BZV55C-5,6V, Diode_SMD:D_SMA, symbol ISM02A-rescue:D_ZENER-MLAB_D
- J1: footprint (none) -> Mlab_Pin_Headers:Straight_2x03
- M1, M2: value HOLE -> HOLE M3; footprint (none) -> Mlab_Mechanical:MountingHole_3mm
- M3, M4: footprint (none) -> Mlab_Mechanical:MountingHole_3mm
Connections:
- net GND: now also C1.2, C2.2, D1.2 (A)
- net VCC renamed +5V
- net +5V: now also C1.1, C2.1, D1.1 (K)
Other:
- note added: "Adjust power voltage range and symbol"
- note added: "Generally a load module has mounting holes connected to the ground."
- note added: "Power source modules has mountig holes floating to avoid ground loops."
